File: Hardware/001000-005.sch (EAGLE design)
At the start: 216 parts, among them IC1 ATSAMD21G18A-AU, IC10 MCP2515T-I_ST, IC11 MCP2515T-I_ST, IC12 CSTCE16M0V53C-R0, IC13 CSTCE16M0V53C-R0, IC14 MPU-6050, IC2 SARA-R410M-02B, IC3 AP2112K-3.3TRG1, IC4 TPS54232D, IC5 TPS563231DRLR, IC6 ATECC508A-MAHDA-T, IC7 SPBTLE-RF, IC8 W25Q16JVZPIQ, IC9 TJA1048TK,118, J1 SF56S006V4BR2000, J2 1040310811, J3 FA1-NCRP-PCB-8, J4 43045-1400, J5 -, J6 FA1-NDRP-PCB-8, J7 M50-3600542R, K1 EE2-3TNU-L, Q1 2N7002DW-7-F, Q2 2N7002,215, Q3 2N7002,215, Q4 2N7002DW-7-F, Q5 BSP76E6433HUMA1, Q6 BSP76E6433HUMA1, Q7 NTR4502PT1G, Q8 BC847CW,115, U1 SN74AVC2T245RSWR, Y1 ABS07-32.768KHZ-1-T

Commit message: -005 board updates
Parts:
- added MCTS, MRTS: PTR1TP06R, testpad:PTR1TP06R
- C46, C47, C48, C49: value GRM1555C1H470JA01D -> 47p
- C55, C56: value GCM155R71C104KA55J -> 100n
- C57: value GRM155R71H222KA01D -> 2n2
- C58: value GCM155R71H103KA55D -> 10n
- R49: value CRCW040228K0FKED -> 28k
- R50: value CRCW040210K2FKED -> 10k2
- R51: value CRCW040240K2FKED -> 40k2
Connections:
- net N$24 renamed MDCD
- net GND: now also R34.2
- net MCTS: now also MCTS.TP; no longer R34.1
- net MRTS: now also MRTS.TP, R34.1; no longer R34.2
Other:
- moved on the sheet: R34
